File: RF_TransimpedanceAmp_FDS02.brd (EAGLE design)
At the start: 69.8 x 38.1 mm, 38 parts, among them IC1 PMA-5452, IC2 PMA-5452, IC3 PMA-5452, IC4 ADM7150ARDZ-3.0, IC5 ADM7150ARDZ-5.0, X1 SMAJ502

Commit message: Misc store point; pushing for work at home
Parts:
- C13, C14, C15, C18, C2, C3: device rlc-jqi:1210 -> rlc-jqi:0805
- moved X1 101.4 mm to (162.5, 61.1)
- moved C13 101.4 mm to (111.0, 66.2)
- moved C2 101.4 mm to (104.6, 66.7)
- moved IC4 101.4 mm to (108.5, 72.3)
- moved C11 101.4 mm to (102.8, 73.5)
- moved C12 101.4 mm to (113.6, 72.9)
- moved C3 101.4 mm to (115.9, 69.5)
- moved C14 38.9 mm to (-6.88, 22.9)
- moved C15 38.9 mm to (-10.3, 33.0)
- moved C16 38.9 mm to (-16.2, 23.4)
- moved C17 38.9 mm to (-13.6, 30.3)
- moved C18 38.9 mm to (-6.86, 28.0)
- moved IC5 38.9 mm to (-13.0, 25.4)
- moved JP1 11.7 mm to (3.17, 15.2), turned to 90 degrees
- moved C8 10.8 mm to (42.4, 35.0)
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Routing:
- net +5V: track 41.2 -> 1.27 mm
- net +15V: track 36.2 -> 0.00 mm
- net +3V: track 61.7 -> 41.9 mm
- net N$4: track 11.9 -> 0.00 mm
- net N$7: track 9.42 -> 4.36 mm
- net RFPD2: track 4.49 -> 1.86 mm
- net RFPD1: track 4.30 -> 1.78 mm
- net N$19: track 2.20 -> 0.00 mm
- net N$14: track 2.18 -> 0.00 mm
Other:
- board size 69.8 x 38.1 mm -> 163.8 x 76.2 mm
